File: HelioHeat/HelioHeat.kicad_pcb (KiCad board)
At the start: 2 copper layers, 2 parts

Commit message: cables
Parts:
- removed REF**: WL-T7DS_0.39INCH, HelioHeatPartsLib:WL-T7DS_0.39INCH
- removed REF**: DFN-8-1EP_2x2mm_P0.5mm_EP0.9x1.5mm, Package_DFN_QFN:DFN-8-1EP_2x2mm_P0.5mm_EP0.9x1.5mm
- added D1: WL-T7DS_0.39INCH_COMMON-ANODE, WL-T7DS_0.39INCH_COMMON-ANODE:WL-T7DS_0.39INCH, F.Cu at (80.5, 27.5)
- added D2: WL-T7DS_0.39INCH_COMMON-ANODE, WL-T7DS_0.39INCH_COMMON-ANODE:WL-T7DS_0.39INCH, F.Cu at (94.5, 27.5)
- added D3: WL-T7DS_0.39INCH_COMMON-ANODE, WL-T7DS_0.39INCH_COMMON-ANODE:WL-T7DS_0.39INCH, F.Cu at (108.0, 27.5)
- added J1: USB_B_Micro, Connector_USB:USB_Micro-B_Amphenol_10103594-0001LF_Horizontal, F.Cu at (133.0, 29.0)
- added R1: 100, Resistor_SMD:R_0201_0603Metric, F.Cu at (87.3, 27.5)
- added R2: 100, Resistor_SMD:R_0201_0603Metric, F.Cu at (101.3, 27.5)
- added R3: 100, Resistor_SMD:R_0201_0603Metric, F.Cu at (114.8, 27.5)
- added U1: ATtiny85-20P, Package_DIP:DIP-8_W7.62mm, F.Cu at (98.2, 52.7)
- added U2: CD4511BE, CD4511BE:DIP794W45P254L1969H508Q16, F.Cu at (79.7, 43.0)
- added U3: CD4511BE, CD4511BE:DIP794W45P254L1969H508Q16, F.Cu at (102.0, 43.0)
- added U4: CD4511BE, CD4511BE:DIP794W45P254L1969H508Q16, F.Cu at (124.7, 43.0)
- added U5: 74HC595, 74HC595:SO16, F.Cu at (85.7, 56.8)
- added U6: 74HC595, 74HC595:SO16, F.Cu at (123.0, 56.0)
- added U7: MCP9700Ax-ELT, Package_TO_SOT_SMD:SOT-353_SC-70-5, F.Cu at (112.0, 58.5)

Commit message: quick adjusment
Parts:
- R1, R2, R3: value 100 -> 220
- moved U7 7.27 mm to (109.0, 51.9)
- moved U5 3.16 mm to (82.7, 55.8), turned to -90 degrees
- moved U1 2.24 mm to (96.2, 51.7)
- moved U6 0.38 mm to (122.8, 56.3), turned to -90 degrees
Connections:
- U1 pad 6: Net-(U1-PB1) -> unconnected-(U1-PB1-Pad6)
- U7 pad 2: GND -> unconnected-(U7-GND-Pad2)
- U7 pad 3: Net-(U1-PB1) -> Net-(U1-PB2)
- U7 pad 4: Net-(U1-PB2) -> +5V

Commit message: fixes
Parts:
- moved U7 23.4 mm to (132.4, 51.4)
- moved U1 23.2 mm to (119.4, 51.4)
- moved U5 16.0 mm to (98.7, 55.8), turned to 90 degrees
- moved U6 13.0 mm to (109.8, 55.8), turned to 90 degrees
Connections:
- U6 pad 4: GND -> unconnected-(U6-QE-Pad4)
- U6 pad 5: GND -> unconnected-(U6-QF-Pad5)
- U6 pad 6: GND -> unconnected-(U6-QG-Pad6)
- U6 pad 7: GND -> unconnected-(U6-QH-Pad7)
- U6 pad 9: GND -> unconnected-(U6-QH&apos;-Pad9)
- U7 pad 2: unconnected-(U7-GND-Pad2) -> GND
