File: HelioHeat/HelioHeat.kicad_pcb (KiCad board)
At the start: 2 copper layers, 14 parts, among them J1 USB_B_Micro, U1 ATtiny85-20P, U2 CD4511BE, U3 CD4511BE, U4 CD4511BE, U5 74HC595, U6 74HC595, U7 MCP9700Ax-ELT

Commit message: i am a routeur
Parts:
- moved U1 25.2 mm to (94.2, 52.7)
- moved U5 14.2 mm to (84.5, 55.5)
- moved U7 10.9 mm to (122.0, 54.5)
Routing:
- net +5V: track 0.00 -> 210.9 mm, vias 0 -> 3
- net GND: track 0.00 -> 185.0 mm, vias 0 -> 3
- net Net-(U5-QH'): track 0.00 -> 45.3 mm
- net Net-(U4-A_OUT): track 0.00 -> 40.9 mm
- net Net-(U1-~{RESET}/PB5): track 0.00 -> 40.2 mm, vias 0 -> 2
- net Net-(U4-D_OUT): track 0.00 -> 38.5 mm
- net Net-(U4-A_IN): track 0.00 -> 38.0 mm
- net Net-(U4-D_IN): track 0.00 -> 35.2 mm
- net Net-(U3-A_IN): track 0.00 -> 34.9 mm
- net Net-(U4-E_OUT): track 0.00 -> 33.8 mm
- net Net-(U1-XTAL1/PB3): track 0.00 -> 30.1 mm
- net Net-(U4-G_OUT): track 0.00 -> 28.3 mm
- net Net-(U2-B_IN): track 0.00 -> 27.3 mm, vias 0 -> 1
- net Net-(U3-E_OUT): track 0.00 -> 25.1 mm
- net Net-(U2-C_IN): track 0.00 -> 24.5 mm, vias 0 -> 1
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Other:
- board outline added: 75.5 x 46 mm
